Commit message: Update_16_02_26

File: Output/Output/URDF/RobiControl.urdf (robot description, URDF)
Before this commit: robot LCAMP_Robot, 13 links, 12 joints
Links:
- link center: mass None -> 50; geometry collision box size=0.3000000142492354 0.14000000059604645 0.06400000303983688; visual box size=0.3000000142492354 0.14000000059604645 0.06400000303983688
- link wheel_hl: mass None -> 50; geometry collision cylinder length=0.028000001329928637 radius=0.04800000227987766; visual cylinder length=0.028000001329928637 radius=0.04800000227987766
- link wheel_hr: mass None -> 50; geometry collision cylinder length=0.028000001329928637 radius=0.04800000227987766; visual cylinder length=0.028000001329928637 radius=0.04800000227987766
- link wheel_vl: mass None -> 50; geometry collision cylinder length=0.028000001329928637 radius=0.04800000227987766; visual cylinder length=0.028000001329928637 radius=0.04800000227987766
- link wheel_vr: mass None -> 50; geometry collision cylinder length=0.028000001329928637 radius=0.04800000227987766; visual cylinder length=0.028000001329928637 radius=0.04800000227987766
