Commit message: Update_01_03_26

File: Output/Output/URDF/Robot_1.urdf (robot description, URDF)
Before this commit: robot LCAMP_Robot, 47 links, 41 joints
Links:
- added link Basplate Pexi; visual mesh filename=.\stlFiles\bodenPlatte_solid.stl scale=0.001 0.001 0.001
- added link CenterPlate Alu; visual mesh filename=.\stlFiles\BasePlate.stl scale=0.001 0.001 0.001
- link Rollers_a_Rollers_a_0_0_33: geometry collision cylinder length=0.01 radius=0.04; visual mesh filename=.\stlFiles\OmniWheel_Roller_2.stl scale=0.001 0.001 0.001
- link Rollers_a_Rollers_a_0_0_7: geometry collision cylinder length=0.01 radius=0.04; visual mesh filename=.\stlFiles\OmniWheel_Roller_2.stl scale=0.001 0.001 0.001
- link Rollers_a_Rollers_a_1_1_35: geometry collision cylinder length=0.01 radius=0.04; visual mesh filename=.\stlFiles\OmniWheel_Roller_2.stl scale=0.001 0.001 0.001
- link Rollers_a_Rollers_a_1_1_9: geometry collision cylinder length=0.01 radius=0.04; visual mesh filename=.\stlFiles\OmniWheel_Roller_2.stl scale=0.001 0.001 0.001
- link Rollers_a_Rollers_a_2_2_11: geometry collision cylinder length=0.01 radius=0.04; visual mesh filename=.\stlFiles\OmniWheel_Roller_2.stl scale=0.001 0.001 0.001
- link Rollers_a_Rollers_a_2_2_37: geometry collision cylinder length=0.01 radius=0.04; visual mesh filename=.\stlFiles\OmniWheel_Roller_2.stl scale=0.001 0.001 0.001
- link Rollers_a_Rollers_a_3_3_13: geometry collision cylinder length=0.01 radius=0.04; visual mesh filename=.\stlFiles\OmniWheel_Roller_2.stl scale=0.001 0.001 0.001
- link Rollers_a_Rollers_a_3_3_39: geometry collision cylinder length=0.01 radius=0.04; visual mesh filename=.\stlFiles\OmniWheel_Roller_2.stl scale=0.001 0.001 0.001
- link Rollers_a_Rollers_a_4_4_15: geometry collision cylinder length=0.01 radius=0.04; visual mesh filename=.\stlFiles\OmniWheel_Roller_2.stl scale=0.001 0.001 0.001
- link Rollers_a_Rollers_a_4_4_41: geometry collision cylinder length=0.01 radius=0.04; visual mesh filename=.\stlFiles\OmniWheel_Roller_2.stl scale=0.001 0.001 0.001
- link Rollers_a_Rollers_a_5_5_17: geometry collision cylinder length=0.01 radius=0.04; visual mesh filename=.\stlFiles\OmniWheel_Roller_2.stl scale=0.001 0.001 0.001
- link Rollers_a_Rollers_a_5_5_43: geometry collision cylinder length=0.01 radius=0.04; visual mesh filename=.\stlFiles\OmniWheel_Roller_2.stl scale=0.001 0.001 0.001
- link Rollers_b_Rollers_b_0_0_19: geometry collision cylinder length=0.01 radius=0.04; visual mesh filename=.\stlFiles\OmniWheel_Roller_2.stl scale=0.001 0.001 0.001
- link Rollers_b_Rollers_b_0_0_45: geometry collision cylinder length=0.01 radius=0.04; visual mesh filename=.\stlFiles\OmniWheel_Roller_2.stl scale=0.001 0.001 0.001
- link Rollers_b_Rollers_b_1_1_21: geometry collision cylinder length=0.01 radius=0.04; visual mesh filename=.\stlFiles\OmniWheel_Roller_2.stl scale=0.001 0.001 0.001
- link Rollers_b_Rollers_b_1_1_47: geometry collision cylinder length=0.01 radius=0.04; visual mesh filename=.\stlFiles\OmniWheel_Roller_2.stl scale=0.001 0.001 0.001
- link Rollers_b_Rollers_b_2_2_23: geometry collision cylinder length=0.01 radius=0.04; visual mesh filename=.\stlFiles\OmniWheel_Roller_2.stl scale=0.001 0.001 0.001
- link Rollers_b_Rollers_b_2_2_49: geometry collision cylinder length=0.01 radius=0.04; visual mesh filename=.\stlFiles\OmniWheel_Roller_2.stl scale=0.001 0.001 0.001
- link Rollers_b_Rollers_b_3_3_25: geometry collision cylinder length=0.01 radius=0.04; visual mesh filename=.\stlFiles\OmniWheel_Roller_2.stl scale=0.001 0.001 0.001
- link Rollers_b_Rollers_b_3_3_51: geometry collision cylinder length=0.01 radius=0.04; visual mesh filename=.\stlFiles\OmniWheel_Roller_2.stl scale=0.001 0.001 0.001
- link Rollers_b_Rollers_b_4_4_27: geometry collision cylinder length=0.01 radius=0.04; visual mesh filename=.\stlFiles\OmniWheel_Roller_2.stl scale=0.001 0.001 0.001
- link Rollers_b_Rollers_b_4_4_53: geometry collision cylinder length=0.01 radius=0.04; visual mesh filename=.\stlFiles\OmniWheel_Roller_2.stl scale=0.001 0.001 0.001
- link Rollers_b_Rollers_b_5_5_29: geometry collision cylinder length=0.01 radius=0.04; visual mesh filename=.\stlFiles\OmniWheel_Roller_2.stl scale=0.001 0.001 0.001
- link Rollers_b_Rollers_b_5_5_55: geometry collision cylinder length=0.01 radius=0.04; visual mesh filename=.\stlFiles\OmniWheel_Roller_2.stl scale=0.001 0.001 0.001
- link _Controller_60a: geometry collision cylinder length=0.01 radius=0.01; visual cylinder length=0.04000000283122063 radius=0.020000001415610313
- link _DC-Drive_1a: geometry collision cylinder length=0.01 radius=0.01; visual box size=0.05000000074505806 0.04500000178813934 0.06400000303983688
- link _DC-Drive_3a: geometry collision cylinder length=0.01 radius=0.01; visual box size=0.05000000074505806 0.04500000178813934 0.06400000303983688
- link _Drive-Holder_31a: geometry collision cylinder length=0.01 radius=0.01; visual cylinder length=0.06000000238418579 radius=0.003000000026077032
- link _Drive-Holder_5a: geometry collision cylinder length=0.01 radius=0.01; visual cylinder length=0.06000000238418579 radius=0.003000000026077032
- link _Omni-Wheel_32a: geometry collision cylinder length=0.01 radius=0.01; visual mesh filename=.\stlFiles\Hub_Cup_8.stl scale=0.001 0.001 0.001
- link _Omni-Wheel_6a: geometry collision cylinder length=0.01 radius=0.01; visual mesh filename=.\stlFiles\Hub_Cup_8.stl scale=0.001 0.001 0.001
- link _Regular-Wheel_2a: geometry collision cylinder length=0.01 radius=0.01; visual mesh filename=.\stlFiles\Hub_Cup_8.stl scale=0.001 0.001 0.001
- link _Regular-Wheel_4a: geometry collision cylinder length=0.01 radius=0.01; visual mesh filename=.\stlFiles\Hub_Cup_8.stl scale=0.001 0.001 0.001
- link _Sensorbox_center_59a: geometry collision cylinder length=0.01 radius=0.01; visual cylinder length=0.04000000283122063 radius=0.020000001415610313
- link _Sensorbox_curved_57a: geometry collision cylinder length=0.01 radius=0.01; visual cylinder length=0.030000001192092896 radius=0.020000001415610313
- link _Sensorbox_curved_58a: geometry collision cylinder length=0.01 radius=0.01; visual cylinder length=0.030000001192092896 radius=0.020000001415610313
Joints:
- removed joint bjoint_Basplate_Pexi
- removed joint bjoint_CenterPlate_Alu
- removed joint bjoint_Drive_bl
- removed joint bjoint_Drive_br
- removed joint bjoint_Drive_fl
- removed joint bjoint_Drive_fr
- removed joint bjoint_Sensorbox_back
- removed joint bjoint_Sensorbox_center
- removed joint bjoint_Sensorbox_controller
- removed joint bjoint_Sensorbox_front
- added joint joint_Basplate Pexi: type fixed, parent center, child Basplate Pexi, origin xyz=0 0 -0.030000001192092896 rpy=0 0 0, axis 0 0 1
- added joint joint_Basplate_Pexi: type fixed, parent center, child Basplate_Pexi, origin xyz=0 0 -0.030000001192092896 rpy=0 0 0, axis 0 0 1
- added joint joint_CenterPlate Alu: type fixed, parent center, child CenterPlate Alu, origin xyz=0 0 0.030000001192092896 rpy=0 0 0, axis 0 0 1
- added joint joint_CenterPlate_Alu: type fixed, parent center, child CenterPlate_Alu, origin xyz=0 0 0.030000001192092896 rpy=0 0 0, axis 0 0 1
- added joint joint_Drive_bl: type fixed, parent center, child Drive_bl, origin xyz=-0.10000000149011612 0.07000000029802322 0 rpy=0 0 0, axis 0 0 1
- added joint joint_Drive_br: type fixed, parent center, child Drive_br, origin xyz=-0.10000000149011612 -0.07000000029802322 0 rpy=0 0 3.1415927410125732, axis 0 0 1
- added joint joint_Drive_fl: type fixed, parent center, child Drive_fl, origin xyz=0.10000000149011612 0.07000000029802322 0 rpy=0 0 0, axis 0 0 1
- added joint joint_Drive_fr: type fixed, parent center, child Drive_fr, origin xyz=0.10000000149011612 -0.07000000029802322 0 rpy=0 0 3.1415927410125732, axis 0 0 1
- added joint joint_Sensorbox_back: type fixed, parent center, child Sensorbox_back, origin xyz=-0.15000000596046448 0 0 rpy=0 0 3.1415927410125732, axis 0 0 1
- added joint joint_Sensorbox_center: type fixed, parent center, child Sensorbox_center, origin xyz=0 -0.07000000029802322 0 rpy=0 0 3.1415927410125732, axis 0 0 1
- added joint joint_Sensorbox_controller: type fixed, parent center, child Sensorbox_controller, origin xyz=0 0.07000000029802322 0 rpy=0 0 0, axis 0 0 1
- added joint joint_Sensorbox_front: type fixed, parent center, child Sensorbox_front, origin xyz=0.15000000596046448 0 0 rpy=0 0 0, axis 0 0 1
