Commit message: Update_03_04_26a

File: Output/URDF/RobiControl.urdf (robot description, URDF)
Before this commit: robot LCAMP_Robot, 31 links, 30 joints
Links:
- removed link Basplate_Pexi
- removed link CenterPlate_Alu
- removed link Drive_bl
- removed link Drive_bl_Regular-Wheel_0
- removed link Drive_bl_Stepper-Drive_0
- removed link Drive_br
- removed link Drive_br_Regular-Wheel_0
- removed link Drive_br_Stepper-Drive_0
- removed link Drive_fl
- removed link Drive_fl_Regular-Wheel_0
- removed link Drive_fl_Stepper-Drive_0
- removed link Drive_fr
- removed link Drive_fr_Regular-Wheel_0
- removed link Drive_fr_Stepper-Drive_0
- removed link Sensorbox_back
- removed link Sensorbox_back_Sensorbox_curved_0
- removed link Sensorbox_center
- removed link Sensorbox_center_Sensor_1_0_13
- removed link Sensorbox_center_Sensor_2_0_15
- removed link Sensorbox_center_Sensorbox_center_0
- removed link Sensorbox_controller
- removed link Sensorbox_controller_Controller_0
- removed link Sensorbox_curved_Sensor_1_0_1
- removed link Sensorbox_curved_Sensor_1_0_7
- removed link Sensorbox_curved_Sensor_2_0_3
- removed link Sensorbox_curved_Sensor_2_0_9
- removed link Sensorbox_curved_Sensor_4_0_11
- removed link Sensorbox_curved_Sensor_4_0_5
- removed link Sensorbox_front
- removed link Sensorbox_front_Sensorbox_curved_0
- added link Wheel1, mass 100; collision cylinder length=0.02 radius=0.01; visual mesh filename=D:\Users\kdRupp\Source\Repos\LCAMP-DHBW\Daten\DHBW CAD-Data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 scale=0.001 0.001 0.001
- added link Wheel2, mass 100; collision cylinder length=0.02 radius=0.01; visual mesh filename=D:\Users\kdRupp\Source\Repos\LCAMP-DHBW\Daten\DHBW CAD-Data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 scale=0.001 0.001 0.001
- added link Wheel3, mass 100; collision cylinder length=0.02 radius=0.01; visual mesh filename=D:\Users\kdRupp\Source\Repos\LCAMP-DHBW\Daten\DHBW CAD-Data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 scale=0.001 0.001 0.001
- added link Wheel4, mass 100; collision cylinder length=0.02 radius=0.01; visual mesh filename=D:\Users\kdRupp\Source\Repos\LCAMP-DHBW\Daten\DHBW CAD-Data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 scale=0.001 0.001 0.001
- added link sbFront, mass 100; collision mesh filename=D:\Users\kdRupp\Source\Repos\LCAMP-DHBW\Daten\DHBW CAD-Data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 scale=0.001 0.001 0.001; visual mesh filename=D:\Users\kdRupp\Source\Repos\LCAMP-DHBW\Daten\DHBW CAD-Data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 scale=0.001 0.001 0.001
- added link sbLeft, mass 100; collision mesh filename=D:\Users\kdRupp\Source\Repos\LCAMP-DHBW\Daten\DHBW CAD-Data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 scale=0.001 0.001 0.001; visual mesh filename=D:\Users\kdRupp\Source\Repos\LCAMP-DHBW\Daten\DHBW CAD-Data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 scale=0.001 0.001 0.001
- added link sbRear, mass 100; collision mesh filename=D:\Users\kdRupp\Source\Repos\LCAMP-DHBW\Daten\DHBW CAD-Data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 scale=0.001 0.001 0.001; visual mesh filename=D:\Users\kdRupp\Source\Repos\LCAMP-DHBW\Daten\DHBW CAD-Data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 scale=0.001 0.001 0.001
- added link sbRight, mass 100; collision mesh filename=D:\Users\kdRupp\Source\Repos\LCAMP-DHBW\Daten\DHBW CAD-Data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 scale=0.001 0.001 0.001; visual mesh filename=D:\Users\kdRupp\Source\Repos\LCAMP-DHBW\Daten\DHBW CAD-Data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 scale=0.001 0.001 0.001
- added link wheel_hl, mass 50; collision cylinder length=0.028000001329928637 radius=0.04800000227987766; visual cylinder length=0.028000001329928637 radius=0.04800000227987766
- added link wheel_hr, mass 50; collision cylinder length=0.028000001329928637 radius=0.04800000227987766; visual cylinder length=0.028000001329928637 radius=0.04800000227987766
- added link wheel_vl, mass 50; collision cylinder length=0.028000001329928637 radius=0.04800000227987766; visual cylinder length=0.028000001329928637 radius=0.04800000227987766
- added link wheel_vr, mass 50; collision cylinder length=0.028000001329928637 radius=0.04800000227987766; visual cylinder length=0.028000001329928637 radius=0.04800000227987766
- link center: mass None -> 50; geometry collision box size=0.3000000142492354 0.14000000059604645 0.06400000303983688; visual box size=0.3000000142492354 0.14000000059604645 0.06400000303983688
Joints:
- removed joint bjoint_Basplate_Pexi
- removed joint bjoint_CenterPlate_Alu
- removed joint bjoint_Drive_bl
- removed joint bjoint_Drive_br
- removed joint bjoint_Drive_fl
- removed joint bjoint_Drive_fr
- removed joint bjoint_Sensorbox_back
- removed joint bjoint_Sensorbox_center
- removed joint bjoint_Sensorbox_controller
- removed joint bjoint_Sensorbox_front
- removed joint j__10b
- removed joint j__12b
- removed joint j__14b
- removed joint j__16b
- removed joint j__2b
- removed joint j__4b
- removed joint j__6b
- removed joint j__8b
- removed joint joint_sub_Drive_bl_Regular-Wheel_0
- removed joint joint_sub_Drive_bl_Stepper-Drive_0
- removed joint joint_sub_Drive_br_Regular-Wheel_0
- removed joint joint_sub_Drive_br_Stepper-Drive_0
- removed joint joint_sub_Drive_fl_Regular-Wheel_0
- removed joint joint_sub_Drive_fl_Stepper-Drive_0
- removed joint joint_sub_Drive_fr_Regular-Wheel_0
- removed joint joint_sub_Drive_fr_Stepper-Drive_0
- removed joint joint_sub_Sensorbox_back_Sensorbox_curved_0
- removed joint joint_sub_Sensorbox_center_Sensorbox_center_0
- removed joint joint_sub_Sensorbox_controller_Controller_0
- removed joint joint_sub_Sensorbox_front_Sensorbox_curved_0
- added joint joint_hl: type continuous, parent center, child wheel_hl, origin xyz=-0.10000000149011612 0.09000000357627869 0 rpy=1.5707963267948966 0 0, axis 0 0 1
- added joint joint_hlhc: type fixed, parent wheel_hl, child Wheel1, origin xyz=0 0 0.012000000104308128 rpy=0 3.141592653589793 0, axis 0 1 0
- added joint joint_hr: type continuous, parent center, child wheel_hr, origin xyz=-0.10000000149011612 -0.09000000357627869 0 rpy=1.5707963267948966 0 0, axis 0 0 1
- added joint joint_hrhc: type fixed, parent wheel_hr, child Wheel2, origin xyz=0 0 -0.012000000104308128 rpy=0 0 0, axis 0 1 0
- added joint joint_sbFront: type fixed, parent center, child sbFront, origin xyz=0.15000000596046448 0 -0.03200000151991844 rpy=0 0 0, axis 0 1 0
- added joint joint_sbLeft: type fixed, parent center, child sbLeft, origin xyz=0 0.07000000029802322 0.03200000151991844 rpy=0 0 0, axis 0 1 0
- added joint joint_sbRear: type fixed, parent center, child sbRear, origin xyz=-0.15000000596046448 0 -0.03200000151991844 rpy=0 0 3.141592653589793, axis 0 1 0
- added joint joint_sbRight: type fixed, parent center, child sbRight, origin xyz=0.1300000101327896 -0.08000000566244125 -0.005000000353902578 rpy=-1.5707963267948966 0 3.141592653589793, axis 0 1 0
- added joint joint_vl: type continuous, parent center, child wheel_vl, origin xyz=0.10000000149011612 0.09000000357627869 0 rpy=1.5707963267948966 0 0, axis 0 0 1
- added joint joint_vlhc: type fixed, parent wheel_vl, child Wheel3, origin xyz=0 0 0.012000000104308128 rpy=0 3.141592653589793 0, axis 0 1 0
- added joint joint_vr: type continuous, parent center, child wheel_vr, origin xyz=0.10000000474974513 -0.09000000357627869 0 rpy=1.5707963267948966 0 0, axis 0 0 1
- added joint joint_vrhc: type fixed, parent wheel_vr, child Wheel4, origin xyz=0 0 -0.012000000104308128 rpy=0 0 0, axis 0 1 0
